Commit message: feat(step4-5): cascade PID controller + diff_drive plugin integration
- Replace gazebo_ros2_control with libgazebo_ros_diff_drive plugin
  * /cmd_vel_wheels (Twist) input, /odom output handled by plugin
  * Eliminates controller_manager dependency in simulation
- Implement cascade PID controller (balance_controller_node.cpp)
  * Outer: velocity loop (cmd_vx vs odom) → theta_setpoint
  * Inner: balance loop (theta_setpoint vs IMU pitch) → wheel v [m/s]
  * Anti-windup PID class, 200 Hz control loop
  * Safety: motor stop when |theta| > 0.35 rad
- Add pause/unpause startup sequence in sim.launch.py
  * Gazebo starts paused (physics frozen)
  * Controller starts at t=2s, unpause_physics at t=3s
  * Prevents robot from falling before controller is ready
- Update pid_params.yaml with tuned initial gains
- Add docs/02_dev_log.md: today's development log
- Update README.md: correct system architecture diagram

Co-Authored-By: Claude Sonnet 4.6 <noreply@anthropic.com>

File: ros2_ws/src/balance_robot_description/urdf/balance_robot.xacro (robot description, xacro)
@@ -4,23 +4,17 @@
        balance_robot.xacro
        Wheeled Inverted Pendulum (2-wheel balance robot)
-       Coordinate convention (REP-103):
-         x: forward,  y: left,  z: up
+       Control: libgazebo_ros_diff_drive (velocity control)
        ======================================================== -->
   <!-- ===================== Properties ====================== -->
-  <!-- Body dimensions -->
-  <xacro:property name="body_mass"   value="1.0"/>
-  <xacro:property name="body_width"  value="0.10"/>   <!-- x (depth) -->
-  <xacro:property name="body_depth"  value="0.08"/>   <!-- y -->
-  <xacro:property name="body_height" value="0.28"/>   <!-- z -->
-  <!-- Wheel dimensions -->
-  <xacro:property name="wheel_mass"   value="0.1"/>
-  <xacro:property name="wheel_radius" value="0.05"/>
-  <xacro:property name="wheel_width"  value="0.02"/>
-  <!-- Body CoM height above wheel axis -->
+  <xacro:property name="body_mass"       value="1.0"/>
+  <xacro:property name="body_width"      value="0.10"/>
+  <xacro:property name="body_depth"      value="0.08"/>
+  <xacro:property name="body_height"     value="0.28"/>
+  <xacro:property name="wheel_mass"      value="0.1"/>
+  <xacro:property name="wheel_radius"    value="0.05"/>
+  <xacro:property name="wheel_width"     value="0.02"/>
   <xacro:property name="body_com_height" value="0.15"/>
-  <!-- Wheel separation (center-to-center along Y) -->
-  <xacro:property name="wheel_sep" value="0.14"/>
+  <xacro:property name="wheel_sep"       value="0.14"/>
   <!-- ===================== Inertia Macros ================== -->
-  <!-- Solid box inertia -->
   <xacro:macro name="box_inertia" params="m w h d">
     <inertial>
@@ -33,9 +27,7 @@
     </inertial>
   </xacro:macro>
-  <!-- Solid cylinder inertia (axis = Y, i.e., wheel spin axis) -->
   <xacro:macro name="cylinder_inertia" params="m r l">
     <inertial>
       <mass value="${m}"/>
-      <!-- ixx/izz: axis perpendicular to cylinder axis -->
       <inertia
         ixx="${(1/12)*m*(3*r*r + l*l)}"
@@ -46,8 +38,5 @@
   </xacro:macro>
   <!-- ===================== Links ============================ -->
-  <!-- World (fixed reference, used only for floating joint workaround) -->
-  <!-- base_footprint: virtual link at ground level -->
   <link name="base_footprint"/>
-  <!-- Base link = chassis body -->
   <link name="base_link">
     <visual>
@@ -66,10 +55,6 @@
       </geometry>
     </collision>
-    <xacro:box_inertia m="${body_mass}"
-                       w="${body_width}"
-                       h="${body_height}"
-                       d="${body_depth}"/>
+    <xacro:box_inertia m="${body_mass}" w="${body_width}" h="${body_height}" d="${body_depth}"/>
   </link>
-  <!-- IMU link (center of body, same as base_link CoM) -->
   <link name="imu_link">
     <visual>
@@ -78,8 +63,6 @@
     </visual>
   </link>
-  <!-- Left wheel -->
   <link name="left_wheel_link">
     <visual>
-      <!-- cylinder default axis is Z; rotate 90° around X to align with Y -->
       <origin xyz="0 0 0" rpy="${pi/2} 0 0"/>
       <geometry>
@@ -96,9 +79,6 @@
       </geometry>
     </collision>
-    <xacro:cylinder_inertia m="${wheel_mass}"
-                            r="${wheel_radius}"
-                            l="${wheel_width}"/>
+    <xacro:cylinder_inertia m="${wheel_mass}" r="${wheel_radius}" l="${wheel_width}"/>
   </link>
-  <!-- Right wheel -->
   <link name="right_wheel_link">
     <visual>
@@ -117,10 +97,7 @@
       </geometry>
     </collision>
-    <xacro:cylinder_inertia m="${wheel_mass}"
-                            r="${wheel_radius}"
-                            l="${wheel_width}"/>
+    <xacro:cylinder_inertia m="${wheel_mass}" r="${wheel_radius}" l="${wheel_width}"/>
   </link>
   <!-- ===================== Joints ========================== -->
-  <!-- base_footprint → base_link (planar joint; robot sits at wheel axis height) -->
   <joint name="base_footprint_joint" type="fixed">
     <parent link="base_footprint"/>
@@ -128,5 +105,4 @@
     <origin xyz="0 0 ${wheel_radius}" rpy="0 0 0"/>
   </joint>
-  <!-- base_link → imu_link (fixed, at body CoM) -->
   <joint name="imu_joint" type="fixed">
     <parent link="base_link"/>
@@ -134,5 +110,4 @@
     <origin xyz="0 0 ${body_com_height}" rpy="0 0 0"/>
   </joint>
-  <!-- base_link → left_wheel (continuous = free rotation around Y) -->
   <joint name="left_wheel_joint" type="continuous">
     <parent link="base_link"/>
@@ -141,7 +116,5 @@
     <axis xyz="0 1 0"/>
     <dynamics damping="0.01" friction="0.1"/>
-    <limit effort="10.0" velocity="10.0"/>
   </joint>
-  <!-- base_link → right_wheel (continuous) -->
   <joint name="right_wheel_joint" type="continuous">
     <parent link="base_link"/>
@@ -150,31 +123,7 @@
     <axis xyz="0 1 0"/>
     <dynamics damping="0.01" friction="0.1"/>
-    <limit effort="10.0" velocity="10.0"/>
   </joint>
-  <!-- ===================== ros2_control ==================== -->
-  <!-- Hardware interface: Gazebo sim -->
-  <ros2_control name="GazeboSystem" type="system">
-    <hardware>
-      <plugin>gazebo_ros2_control/GazeboSystem</plugin>
-    </hardware>
-    <joint name="left_wheel_joint">
-      <command_interface name="effort">
-        <param name="min">-10</param>
-        <param name="max"> 10</param>
-      </command_interface>
-      <state_interface name="position"/>
-      <state_interface name="velocity"/>
-    </joint>
-    <joint name="right_wheel_joint">
-      <command_interface name="effort">
-        <param name="min">-10</param>
-        <param name="max"> 10</param>
-      </command_interface>
-      <state_interface name="position"/>
-      <state_interface name="velocity"/>
-    </joint>
-  </ros2_control>
   <!-- ===================== Gazebo Plugins ================== -->
-  <!-- IMU sensor plugin -->
+  <!-- IMU sensor -->
   <gazebo reference="imu_link">
     <sensor name="imu_sensor" type="imu">
@@ -202,24 +151,35 @@
     </sensor>
   </gazebo>
-  <!-- gazebo_ros2_control plugin -->
+  <!-- Differential drive controller
+       Subscribes to /cmd_vel_wheels → drives left/right wheel joints
+       Publishes  /odom              → odometry for velocity feedback   -->
   <gazebo>
-    <plugin name="gazebo_ros2_control" filename="libgazebo_ros2_control.so">
-      <robot_sim_type>gazebo_ros2_control/GazeboSystem</robot_sim_type>
-      <parameters>$(find balance_robot_gazebo)/config/ros2_control.yaml</parameters>
+    <plugin name="differential_drive_controller" filename="libgazebo_ros_diff_drive.so">
+      <ros>
+        <remapping>cmd_vel:=cmd_vel_wheels</remapping>
+        <remapping>odom:=odom</remapping>
+      </ros>
+      <left_joint>left_wheel_joint</left_joint>
+      <right_joint>right_wheel_joint</right_joint>
+      <wheel_separation>${wheel_sep}</wheel_separation>
+      <wheel_diameter>${2*wheel_radius}</wheel_diameter>
+      <max_wheel_torque>20</max_wheel_torque>
+      <max_wheel_acceleration>10</max_wheel_acceleration>
+      <publish_odom>true</publish_odom>
+      <publish_odom_tf>true</publish_odom_tf>
+      <publish_wheel_tf>false</publish_wheel_tf>
+      <odometry_frame>odom</odometry_frame>
+      <robot_base_frame>base_footprint</robot_base_frame>
     </plugin>
   </gazebo>
-  <!-- Wheel friction (Gazebo material) -->
+  <!-- Wheel friction -->
   <gazebo reference="left_wheel_link">
-    <mu1>1.0</mu1>
-    <mu2>1.0</mu2>
-    <kp>1e6</kp>
-    <kd>100</kd>
+    <mu1>1.0</mu1><mu2>1.0</mu2>
+    <kp>1e6</kp><kd>100</kd>
     <material>Gazebo/DarkGrey</material>
   </gazebo>
   <gazebo reference="right_wheel_link">
-    <mu1>1.0</mu1>
-    <mu2>1.0</mu2>
-    <kp>1e6</kp>
-    <kd>100</kd>
+    <mu1>1.0</mu1><mu2>1.0</mu2>
+    <kp>1e6</kp><kd>100</kd>
     <material>Gazebo/DarkGrey</material>
   </gazebo>
